File: usb_msc/usb_msc.kicad_sch (KiCad schematic)
At the start: 56 parts, among them J1 Micro_SD_Card_Det_Hirose_DM3D, J2 USB_C_Receptacle_USB2.0, J3 USB_B_Micro, SW1 SW_Push, U1 STM32F730R8Tx, U2 USB3318, U3 AP7313-33SR, Y1 ABM8-13.000MHZ-10-1-U-T

Commit message: add schematics as pdf
Other:
- note added: "USB3318 required 13MHz STM32 DFU requires 4..26MHz XTAL lower is better"
- note removed: "DFU requires 4..26MHz XTAL lower is better"
- note removed: "f_MAX_SDMMC: 50MHz (48MHz?)"
- company: (none) -> znuh
- title: (none) -> usb_msc devboard
Changed lines of the file:
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@@
 (kicad_sch (version 20230121) (generator eeschema)
   (paper "A4")
+  (title_block
+    (title "usb_msc devboard")
+    (date "2023-03-19")
+    (rev "v1")
+    (company "znuh")
+  )
   (junction (at 54.61 44.45) (diameter 0) (color 0 0 0 0)
   )
@@
     (effects (font (size 1.27 1.27) (thickness 0.254) bold) (justify left bottom))
   )
-  (text "DFU requires 4..26MHz XTAL\nlower is better" (at 252.73 172.72 0)
+  (text "USB3318 required 13MHz\nSTM32 DFU requires 4..26MHz XTAL\nlower is better"
+    (at 139.7 71.12 0)
     (effects (font (size 1.27 1.27)) (justify left bottom))
   )
-  (text "f_MAX_SDMMC: 50MHz (48MHz?)" (at 213.36 175.26 0)
-    (effects (font (size 1.27 1.27)) (justify left bottom))
-  )
